File: Plate_Mid/Unison_Plate_Mid.kicad_pcb (KiCad board)
At the start: 2 copper layers, 285 x 95.1 mm, 295 parts, among them J1 USB4085-GF-A_REVA, U1 ATmega32U4-AU, Y1 16MHz

Commit message: Update: v04基板を元に、Eco1.Userレイヤーにプレート用データを作成。
Parts:
- removed ? (x36): , mx2u:M2_Hole
- removed OL1: OLED, ukiha:OLED_rev2
- removed the REF** at (159.5, 63.6)
- added H1: MountingHole, ukiha:M2_Hole, F.Cu at (20.6, 33.5)
- added H10: MountingHole, ukiha:M2_Hole, F.Cu at (300.6, 37.2)
- added H11: MountingHole, ukiha:M2_Hole, F.Cu at (20.6, 57.6)
- added H12: MountingHole, ukiha:M2_Hole, F.Cu at (160.6, 57.6)
- added H13: MountingHole, ukiha:M2_Hole, F.Cu at (300.6, 57.6)
- added H14: MountingHole, ukiha:M2_Hole, F.Cu at (20.6, 123.5)
- added H15: MountingHole, ukiha:M2_Hole, F.Cu at (160.6, 123.5)
- added H16: MountingHole, ukiha:M2_Hole, F.Cu at (300.6, 123.5)
- added H17: MountingHole, ukiha:M2_Hole, F.Cu at (103.4, 123.5)
- added H18: MountingHole, ukiha:M2_Hole, F.Cu at (200.6, 123.5)
- added H2: MountingHole, ukiha:M2_Hole, F.Cu at (113.0, 33.5)
- added H3: MountingHole, ukiha:M2_Hole, F.Cu at (160.6, 33.5)
- added H4: MountingHole, ukiha:M2_Hole, F.Cu at (208.2, 33.5)
- added H5: MountingHole, ukiha:M2_Hole, F.Cu at (300.6, 33.5)
- added H6: MountingHole, ukiha:M2_Hole, F.Cu at (20.6, 37.2)
- added H7: MountingHole, ukiha:M2_Hole, F.Cu at (113.0, 37.2)
- added H8: MountingHole, ukiha:M2_Hole, F.Cu at (160.6, 37.2)
- added H9: MountingHole, ukiha:M2_Hole, F.Cu at (208.2, 37.2)
- added J2: Conn_02x05[3_Odd_Even, Connector_PinHeader_2.54mm:PinHeader_2x03_P2.54mm_Vertical, B.Cu at (140.4, 59.2)
- added J3: LED Shade, Connector_PinSocket_2.54mm:PinSocket_1x03_P2.54mm_Vertical, F.Cu at (76.6, 34.8)
- added J4: Conn_01x02, Connector_PinHeader_2.54mm:PinHeader_1x02_P2.54mm_Vertical, B.Cu at (120.7, 36.1)
- added JP_LED1: SolderJumper_3_Open, Jumper:SolderJumper-3_P1.3mm_Open_Pad1.0x1.5mm_NumberLabels, B.Cu at (95.9, 37.2)
- added L9: SK6812MINI, LED_SMD:LED_SK6812MINI_PLCC4_3.5x3.5mm_P1.75mm, F.Cu at (268.5, 37.2)
- added REF**: 60_Outline, #local:60_Outline-TinyHole_No_Hole3, F.Cu at (160.6, 78.7)
- added SW_60_3: SW_Push, ukiha:MXOnly-2U-NoLED_16mm, F.Cu at (202.6, 117.8)
- added SW_70_2: SW_Push, ukiha:CherryMX_MidHeight_16mm_rev2_merged_hole_1.5u_guide, F.Cu at (232.0, 117.8)
- added SW_80_2: SW_Push, ukiha:CherryMX_MidHeight_16mm_rev2_merged_hole_1.5u_guide, F.Cu at (257.2, 117.8)
- L1, L2, L3, L4, L5, L6, L7, L8: value YS_SK6812MINI_E_modify_GND_powerInput -> SK6812MINI; footprint mx2u:YS-SK6812MINI-E -> LED_SMD:LED_SK6812MINI_PLCC4_3.5x3.5mm_P1.75mm
- SW_10_1, SW_12_1, SW_12_2, SW_13_1, SW_13_2, SW_14, SW_15, SW_16, SW_17_1, SW_19_1, SW_20_1, SW_23_1, SW_23_2, SW_24_1, SW_25_1, SW_26, SW_27_1, SW_27_2, SW_28_1, SW_28_2, SW_29, SW_30_1, SW_31, SW_32_1, SW_32_2, SW_34, SW_36_1, SW_36_2, SW_37_1, SW_38_1, SW_39_1, SW_40_1, SW_41_1, SW_41_2, SW_42, SW_43, SW_46_1, SW_46_2, SW_47, SW_48, SW_49, SW_50, SW_51_1, SW_51_2, SW_52, SW_54, SW_56, SW_57, SW_58, SW_59, SW_6, SW_60_1, SW_61, SW_62, SW_63, SW_64, SW_67, SW_68, SW_69, SW_70_1, SW_71, SW_72_1, SW_73_1, SW_74, SW_76, SW_78_1, SW_78_2, SW_79, SW_7_1, SW_80_1, SW_81, SW_82_1, SW_82_2, SW_83_1, SW_83_2, SW_84, SW_85_1, SW_86, SW_87_1, SW_87_2, SW_89, SW_9, SW_90_1, SW_94, SW_95, SW_96, SW_97_1, SW_97_2, SW_98_1, SW_98_2: footprint ukiha:CherryMX_MidHeight_16mm_rev2 -> ukiha:CherryMX_MidHeight_16mm_rev2_merged_hole
- SW_10_2, SW_19_2, SW_35_2, SW_39_2, SW_45_2, SW_75_3, SW_85_2: footprint ukiha:CherryMX_MidHeight_16mm_rev2_2u_guide -> ukiha:CherryMX_MidHeight_16mm_rev2_merged_hole_2u_guide
- SW_17_2, SW_18_2, SW_20_2, SW_25_3, SW_30_2, SW_35_3, SW_38_2, SW_45_3, SW_45_4, SW_65_2, SW_65_3, SW_72_2, SW_73_2, SW_7_2, SW_85_3, SW_8_2: footprint ukiha:CherryMX_MidHeight_16mm_rev2_1.5u_guide -> ukiha:CherryMX_MidHeight_16mm_rev2_merged_hole_1.5u_guide
- SW_18_1, SW_21, SW_53, SW_8_1, SW_91: footprint ukiha:CherryMX_MidHeight_16mm_rev2 -> ukiha:MXOnly-1U-NoLED_16mm
- SW_25_2, SW_60_2, SW_90_2: footprint ukiha:CherryMX_MidHeight_16mm_rev2_2U_vertical_guide -> ukiha:CherryMX_MidHeight_16mm_rev2_merged_hole_2U_vertical_guide
- SW_35_1, SW_45_1, SW_65_1: footprint ukiha:CherryMX_MidHeight_16mm_rev2 -> ukiha:CherryMX_MidHeight_16mm_rev2_merged_hole_2u_guide
- SW_37_2: footprint ukiha:CherryMX_MidHeight_16mm_rev2_1.5u_alt_guide -> ukiha:CherryMX_MidHeight_16mm_rev2_merged_hole_1.5u_alt_guide
- SW_75_1: footprint ukiha:CherryMX_MidHeight_16mm_rev2 -> ukiha:MXOnly-2U-NoLED_16mm
- SW_75_2: footprint ukiha:CherryMX_MidHeight_16mm_rev2_1.5u_guide -> ukiha:MXOnly-1.5U-NoLED_16mm
- U1: value ATmega32U4-AU -> ATmega32U4-MU; footprint keebio:ATMEGA32U4-AU -> swanmatch:QFN-44-1EP_7x7mm_Pitch0.5mm
- moved L4 53.7 mm to (100.5, 37.2), turned to 270 degrees
- moved L5 35.8 mm to (134.1, 37.2), turned to 270 degrees
- moved L6 35.8 mm to (167.7, 37.2), turned to 270 degrees
- moved L7 35.8 mm to (201.3, 37.2), turned to 270 degrees
- moved L8 35.8 mm to (234.9, 37.2), turned to 270 degrees
- moved L3 34.1 mm to (50.1, 37.2), turned to 270 degrees
- moved D26 22.4 mm to (84.8, 47.1)
- moved R1 19.6 mm to (31.4, 43.0)
- moved D2 19.3 mm to (24.6, 39.4), turned to 0 degrees
- moved D90 18.9 mm to (266.1, 49.5)
- moved D70 18.8 mm to (212.6, 112.8)
- moved D88 18.5 mm to (269.6, 112.8)
- moved C1 17.0 mm to (123.4, 65.6), turned to 90 degrees
- moved D76 16.1 mm to (219.0, 112.8)
- moved L2 15.9 mm to (80.6, 37.2), turned to 270 degrees
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Other:
- outline, holes or cut-outs redrawn
- board text added: "JLCJLCJLCJLC"
- board text added: "MISO SCK RST"
- board text added: "Unison"
- board text added: "VCC MOSI GND"
- board text added: "v04_MU @jpskenn"
- board text removed: "Unison Mid Plate(A) v03 @jpskenn"
