File: Plate_Mid_OP-1/Unison_Plate_Mid.kicad_pcb (KiCad board)
At the start: 2 copper layers, 285 x 28.8 mm, 6 parts

Commit message: Update: OP-1スタイルのミドルプレートをv04で作成。
Parts:
- moved ? 0.30 mm to (159.6, 42.9)
- moved ? 0.30 mm to (299.6, 42.9)
- moved ? 0.30 mm to (19.6, 42.9)
- moved ? 0.05 mm to (159.6, 18.8)
- moved ? 0.05 mm to (299.6, 18.8)
- moved ? 0.05 mm to (19.6, 18.8)
Other:
- board size 285 x 28.8 mm -> 285 x 28.5 mm
- board text added: "Unison Mid Plate(A) v04 @jpskenn"
- board text removed: "Unison Mid Plate(A) v03 @jpskenn"
